Commit message: change urata_hrpsys_config parameters

File: hrpsys_ros_bridge_tutorials/models/JAXON_RED.urdf.xacro (robot description, xacro)
@@ -60,5 +60,8 @@
     <!-- <origin xyz="0.097542410 -0.000296955 0.063307448" rpy="-0.007600616 0.046755703 -0.015569626" /> -->
     <!-- 2016.6.1 tamura kumagai by modification of mount frame -->
-    <origin rpy="-0.005 0.048 -0.020569626" xyz="0.095 0.003596955 0.075307448"/>
+    <!-- <origin rpy="-0.005 0.048 -0.020569626" xyz="0.095 0.003596955 0.075307448"/> -->
+    <!-- 2020.10.23 copy new head parameter from JAXON.urdf.xacro -->
+    <!-- <origin rpy="0.01 0.245 0.03" xyz="0.12 -0.025 0.09"/> -->
+    <origin rpy="0.003 0.255 -0.02" xyz="0.1 0.01 0.085"/>
   </joint>
   <!-- for calibration / original offset of camera_frame
